Commit message: PNP rviz complete

File: install/arm_urdf/share/arm_urdf/urdf/arm_urdf.xacro (robot description, xacro)
@@ -287,4 +287,11 @@
         </collision>
     </link>
+    <link name="grasp_frame">
+    </link>
+    <joint name="link6_to_grasp_frame" type="fixed">
+    <parent link="link6"/>
+    <child link="grasp_frame"/>
+    <origin xyz="-0.06 0.1 -0.025" rpy="1.5708 0 -1.5708"/> <!-- adjust based on actual offset -->
+    </joint>
     <joint name="base_footprint_joint" type="fixed">
         <parent link="base_footprint" />

File: install/arm_urdf_moveit_config/share/arm_urdf_moveit_config/config/arm_urdf.ros2_control.xacro (robot description, xacro)
@@ -8,4 +8,11 @@
                 <plugin>mock_components/GenericSystem</plugin>
             </hardware>
+            <joint name="AX_12A_04_Revolute-34">
+                <command_interface name="position"/>
+                <state_interface name="position">
+                  <param name="initial_value">${initial_positions['AX_12A_04_Revolute-34']}</param>
+                </state_interface>
+                <state_interface name="velocity"/>
+            </joint>
             <joint name="base_link_link1_to_base_link">
                 <command_interface name="position"/>
@@ -50,11 +57,4 @@
                 <state_interface name="velocity"/>
             </joint>
-            <joint name="AX_12A_04_Revolute-34">
-                <command_interface name="position"/>
-                <state_interface name="position">
-                  <param name="initial_value">${initial_positions['AX_12A_04_Revolute-34']}</param>
-                </state_interface>
-                <state_interface name="velocity"/>
-            </joint>
         </ros2_control>
     </xacro:macro>

Commit message: Motor meshes added

File: install/arm_urdf/share/arm_urdf/urdf/arm_urdf.xacro (robot description, xacro)
@@ -39,4 +39,20 @@
             </geometry>
         </collision>
+        <!-- Motor geometry -->
+        <visual>
+            <origin xyz="0 0.05 0.02" rpy="1.57 0 0" />
+            <geometry>
+            <cylinder radius="0.02" length="0.1"/>
+            </geometry>
+            <material name="gray">
+            <color rgba="0.0 0.0 1.0 1.0"/>
+            </material>
+        </visual>
+        <collision>
+            <origin xyz="0 0.05 0.02" rpy="0 0 0"/>
+            <geometry>
+            <cylinder radius="0.02" length="0.1"/>
+            </geometry>
+        </collision>
     </link>
     <link name="link2">
@@ -56,4 +72,20 @@
             <geometry>
                 <mesh filename="file://$(find arm_urdf)/meshes/link2.stl" scale="0.001 0.001 0.001" />
+            </geometry>
+        </collision>
+          <!-- Motor geometry -->
+        <visual>
+            <origin xyz="-0.02 0.02 -0.12" rpy="0.0 1.7 1.57"/>
+            <geometry>
+            <box size="0.08 0.05 0.04"/>
+            </geometry>
+            <material name="dark_gray">
+            <color rgba="0.0 0.0 1.0 1.0"/>
+            </material>
+        </visual>
+        <collision>
+            <origin xyz="-0.02 0.02 -0.12" rpy="0.0 1.7 1.57"/>
+            <geometry>
+            <box size="0.08 0.05 0.04"/>
             </geometry>
         </collision>
