Commit message: Gazebo Working

File: src/arm_urdf/urdf/arm_urdf.xacro (robot description, xacro)
@@ -1,4 +1,9 @@
 <?xml version='1.0' encoding='utf-8'?>
 <robot name="arm_urdf" xmlns:xacro="http://www.ros.org/wiki/xacro">
+    <link name = "world"/>
+    <joint name="base_to_world" type="fixed">
+        <parent link="world" />
+        <child link="base_footprint" />
+    </joint>
     <link name="base_footprint" />
     <link name="base_link">
@@ -41,5 +46,5 @@
         <!-- Motor geometry -->
         <visual>
-            <origin xyz="0 0.05 0.02" rpy="1.57 0 0" />
+            <origin xyz="0 0.05 0.04" rpy="1.57 0 0" />
             <geometry>
             <cylinder radius="0.02" length="0.1"/>
@@ -50,5 +55,5 @@
         </visual>
         <collision>
-            <origin xyz="0 0.05 0.02" rpy="0 0 0"/>
+            <origin xyz="0 0.05 0.04" rpy="0 0 0"/>
             <geometry>
             <cylinder radius="0.02" length="0.1"/>
@@ -365,5 +370,5 @@
         <child link="Gear_Flange_Driven" />
         <axis xyz="0.091609 0.2724359999999999 0.957803" />
-        <mimic joint="AX_12A_04_Revolute-34" multiplier="1.0" offset="0"/>
+        <!-- <mimic joint="AX_12A_04_Revolute-34" multiplier="1.0" offset="0"/> -->
     </joint>
     <joint name="Gear_Flange_Driven_Rigid-25" type="fixed">

File: src/arm_urdf_moveit_config/config/arm_urdf.ros2_control.xacro (robot description, xacro)
@@ -3,16 +3,15 @@
     <xacro:macro name="arm_urdf_ros2_control" params="name initial_positions_file">
         <xacro:property name="initial_positions" value="${load_yaml(initial_positions_file)['initial_positions']}"/>
-        <ros2_control name="${name}" type="system">
+      <gazebo>
+        <plugin name="gazebo_ros2_control" filename="libgazebo_ros2_control.so">
+            <update_rate>1000</update_rate>
+            <parameters>$(find arm_urdf_moveit_config)/config/ros2_controllers.yaml</parameters>
+        </plugin>
+      </gazebo>
+        <ros2_control name="GazeboSimSystem" type="system">
             <hardware>
                 <!-- By default, set up controllers for simulation. This won't work on real hardware -->
-                <plugin>mock_components/GenericSystem</plugin>
+                <plugin>gazebo_ros2_control/GazeboSystem</plugin>
             </hardware>
-            <joint name="AX_12A_04_Revolute-34">
-                <command_interface name="position"/>
-                <state_interface name="position">
-                  <param name="initial_value">${initial_positions['AX_12A_04_Revolute-34']}</param>
-                </state_interface>
-                <state_interface name="velocity"/>
-            </joint>
             <joint name="base_link_link1_to_base_link">
                 <command_interface name="position"/>
@@ -57,4 +56,18 @@
                 <state_interface name="velocity"/>
             </joint>
+            <joint name="link6_Revolute-24">
+                <command_interface name="position"/>
+                <state_interface name="position">
+                  <param name="initial_value">${initial_positions['link6_Revolute-24']}</param>
+                </state_interface>
+                <state_interface name="velocity"/>
+            </joint>
+            <joint name="AX_12A_04_Revolute-34">
+                <command_interface name="position"/>
+                <state_interface name="position">
+                  <param name="initial_value">${initial_positions['AX_12A_04_Revolute-34']}</param>
+                </state_interface>
+                <state_interface name="velocity"/>
+            </joint>
         </ros2_control>
     </xacro:macro>
