Commit message: Setup issue resolved

File: src/arm_urdf/urdf/arm_urdf.urdf (robot description, URDF)
Before this commit: robot arm_urdf, 15 links, 14 joints
Links:
- link AX_12A_01: geometry collision mesh filename=package://arm_urdf/meshes/AX_12A_01.stl scale=0.001 0.001 0.001; visual mesh filename=package://arm_urdf/meshes/AX_12A_01.stl scale=0.001 0.001 0.001
- link AX_12A_02: geometry collision mesh filename=package://arm_urdf/meshes/AX_12A_02.stl scale=0.001 0.001 0.001; visual mesh filename=package://arm_urdf/meshes/AX_12A_02.stl scale=0.001 0.001 0.001
- link AX_12A_03: geometry collision mesh filename=package://arm_urdf/meshes/AX_12A_03.stl scale=0.001 0.001 0.001; visual mesh filename=package://arm_urdf/meshes/AX_12A_03.stl scale=0.001 0.001 0.001
- link AX_12A_04: geometry collision mesh filename=package://arm_urdf/meshes/AX_12A_04.stl scale=0.001 0.001 0.001; visual mesh filename=package://arm_urdf/meshes/AX_12A_04.stl scale=0.001 0.001 0.001
- link Gear_Flange_Driven: geometry collision mesh filename=package://arm_urdf/meshes/Gear_Flange_Driven.stl scale=0.001 0.001 0.001; visual mesh filename=package://arm_urdf/meshes/Gear_Flange_Driven.stl scale=0.001 0.001 0.001
- link Gear_Flange_Motor: geometry collision mesh filename=package://arm_urdf/meshes/Gear_Flange_Motor.stl scale=0.001 0.001 0.001; visual mesh filename=package://arm_urdf/meshes/Gear_Flange_Motor.stl scale=0.001 0.001 0.001
- link Soft_finger_1: geometry collision mesh filename=package://arm_urdf/meshes/Soft_finger_1.stl scale=0.001 0.001 0.001; visual mesh filename=package://arm_urdf/meshes/Soft_finger_1.stl scale=0.001 0.001 0.001
- link Soft_finger_2: geometry collision mesh filename=package://arm_urdf/meshes/Soft_finger_2.stl scale=0.001 0.001 0.001; visual mesh filename=package://arm_urdf/meshes/Soft_finger_2.stl scale=0.001 0.001 0.001
- link base_link: geometry collision mesh filename=package://arm_urdf/meshes/base_link.stl scale=0.001 0.001 0.001; visual mesh filename=file://$(find arm_urdf)/meshes/base_link.stl scale=0.001 0.001 0.001
- link link1: geometry collision mesh filename=package://arm_urdf/meshes/link1.stl scale=0.001 0.001 0.001; visual mesh filename=package://arm_urdf/meshes/link1.stl scale=0.001 0.001 0.001
- link link2: geometry collision mesh filename=package://arm_urdf/meshes/link2.stl scale=0.001 0.001 0.001; visual mesh filename=package://arm_urdf/meshes/link2.stl scale=0.001 0.001 0.001
- link link3: geometry collision mesh filename=package://arm_urdf/meshes/link3.stl scale=0.001 0.001 0.001; visual mesh filename=package://arm_urdf/meshes/link3.stl scale=0.001 0.001 0.001
- link link4: geometry collision mesh filename=package://arm_urdf/meshes/link4.stl scale=0.001 0.001 0.001; visual mesh filename=package://arm_urdf/meshes/link4.stl scale=0.001 0.001 0.001
- link link5: geometry collision mesh filename=package://arm_urdf/meshes/link5.stl scale=0.001 0.001 0.001; visual mesh filename=package://arm_urdf/meshes/link5.stl scale=0.001 0.001 0.001
- link link6: geometry collision mesh filename=package://arm_urdf/meshes/link6.stl scale=0.001 0.001 0.001; visual mesh filename=package://arm_urdf/meshes/link6.stl scale=0.001 0.001 0.001

File: src/arm_urdf/urdf/arm_urdf.xacro (robot description, xacro)
@@ -324,5 +324,5 @@
     <parent link="link6"/>
     <child link="grasp_frame"/>
-    <origin xyz="-0.06 0.1 -0.025" rpy="1.5708 0 -1.5708"/> <!-- adjust based on actual offset -->
+    <origin xyz="-0.06 0.1 -0.025" rpy="1.5708 0 -1.5708"/>
     </joint>
     <joint name="base_footprint_joint" type="fixed">
